Commit message: Feature/Set robot_sn as default prefix to the robot joint and link names (#45)

File: flexiv_description/urdf/rizon.urdf.xacro (robot description, xacro)
@@ -1,6 +1,4 @@
 <?xml version="1.0" encoding="utf-8"?>
-<robot xmlns:xacro="http://www.ros.org/wiki/xacro" name="$(arg name)">
-  <!-- Enable setting arguments from the launch file -->
-  <xacro:arg name="name" default="rizon"/>
+<robot xmlns:xacro="http://www.ros.org/wiki/xacro" name="rizon">
   <!-- 'rizon_type' values: rizon4, rizon4s, rizon10, rizon10s -->
   <xacro:arg name="rizon_type" default="rizon4"/>
@@ -8,5 +6,5 @@
   <xacro:include filename="$(find flexiv_description)/urdf/rizon_macro.xacro"/>
   <!-- parameters -->
-  <xacro:arg name="prefix" default="" />
+  <xacro:arg name="arm_prefix" default="" />
   <xacro:arg name="robot_sn" default="" />
   <xacro:arg name="load_gripper" default="false" />
@@ -14,16 +12,12 @@
   <xacro:arg name="use_fake_hardware" default="false" />
   <xacro:arg name="fake_sensor_commands" default="false" />
-  <xacro:arg name="initial_positions_file" default="$(find flexiv_description)/config/initial_positions.yaml"/>
-  <!-- convert to property to use substitution in function -->
-  <xacro:property name="initial_positions_file" default="$(arg initial_positions_file)"/>
   <xacro:rizon_robot
     rizon_type="$(arg rizon_type)"
-    prefix="$(arg prefix)"
+    arm_prefix="$(arg arm_prefix)"
     robot_sn="$(arg robot_sn)"
     load_gripper="$(arg load_gripper)"
     gripper_name="$(arg gripper_name)"
     use_fake_hardware="$(arg use_fake_hardware)"
-    fake_sensor_commands="$(arg fake_sensor_commands)"
-    initial_positions="${xacro.load_yaml(initial_positions_file)}">
+    fake_sensor_commands="$(arg fake_sensor_commands)">
   </xacro:rizon_robot>
 </robot>

File: flexiv_description/urdf/rizon_macro.xacro (robot description, xacro)
@@ -1,7 +1,8 @@
 <?xml version="1.0"?>
 <robot xmlns:xacro="http://wiki.ros.org/xacro">
-  <xacro:macro name="rizon_robot" params="
+  <xacro:macro name="rizon_robot"
+    params="
     rizon_type
-    prefix
+    arm_prefix
     robot_sn
     load_gripper:=false
@@ -9,6 +10,7 @@
     use_fake_hardware:=false
     fake_sensor_commands:=false
-    initial_positions:=${dict(joint1=0.0,joint2=-0.69813,joint3=0.0,joint4=1.570796,joint5=0.0,joint6=0.69813,joint7=0.0)}
     ">
+    <!-- Prefix defaults to 'arm_prefix_robot_sn' -->
+    <xacro:property name="prefix" value="${arm_prefix + robot_sn + '_'}" />
     <!-- Load gripper -->
     <xacro:if value="${load_gripper and gripper_name=='Flexiv-GN01'}">
@@ -21,24 +23,24 @@
     <xacro:if value="${rizon_type=='rizon4' or rizon_type=='rizon4s'}">
       <xacro:include filename="$(find flexiv_description)/urdf/rizon4_joints_links.xacro" />
-      <xacro:rizon4_joints_links rizon_type="${rizon_type}" prefix="${prefix}" mesh_prefix_path="package://flexiv_description/" />
+      <xacro:rizon4_joints_links rizon_type="${rizon_type}" prefix="${prefix}"
+        mesh_prefix_path="package://flexiv_description/" />
       <!-- ros2 control include -->
-      <xacro:include filename="$(find flexiv_description)/urdf/rizon4.ros2_control.xacro"/>
+      <xacro:include filename="$(find flexiv_description)/urdf/rizon4.ros2_control.xacro" />
       <xacro:rizon4_ros2_control prefix="${prefix}" robot_sn="${robot_sn}"
         use_fake_hardware="${use_fake_hardware}"
         fake_sensor_commands="${fake_sensor_commands}"
-        initial_positions="${initial_positions}"
-        />
+      />
     </xacro:if>
     <!-- Rizon 10 or 10s-->
     <xacro:if value="${rizon_type=='rizon10' or rizon_type=='rizon10s'}">
       <xacro:include filename="$(find flexiv_description)/urdf/rizon10_joints_links.xacro" />
-      <xacro:rizon10_joints_links rizon_type="${rizon_type}" prefix="${prefix}" mesh_prefix_path="package://flexiv_description/" />
+      <xacro:rizon10_joints_links rizon_type="${rizon_type}" prefix="${prefix}"
+        mesh_prefix_path="package://flexiv_description/" />
       <!-- ros2 control include -->
-      <xacro:include filename="$(find flexiv_description)/urdf/rizon10.ros2_control.xacro"/>
+      <xacro:include filename="$(find flexiv_description)/urdf/rizon10.ros2_control.xacro" />
       <xacro:rizon10_ros2_control prefix="${prefix}" robot_sn="${robot_sn}"
         use_fake_hardware="${use_fake_hardware}"
         fake_sensor_commands="${fake_sensor_commands}"
-        initial_positions="${initial_positions}"
-        />
+      />
     </xacro:if>
   </xacro:macro>

File: flexiv_moveit_config/srdf/grav.srdf.xacro (robot description, xacro)
@@ -1,6 +1,8 @@
 <?xml version="1.0" encoding="UTF-8"?>
 <robot xmlns:xacro="http://www.ros.org/wiki/xacro">
-    <xacro:macro name="grav_srdf" params="name prefix">
-        <group name="${prefix}grav_gripper">
+    <xacro:macro name="grav_srdf" params="arm_prefix robot_sn">
+        <!-- Prefix defaults to 'arm_prefix_robot_sn' -->
+        <xacro:property name="prefix" value="${arm_prefix + robot_sn + '_'}" />
+        <group name="grav_gripper">
             <joint name="${prefix}gripper_base_joint" />
             <joint name="${prefix}open_fingers_tcp_joint" />
@@ -24,11 +26,12 @@
         <passive_joint name="${prefix}right_inner_knuckle_joint" />
         <passive_joint name="${prefix}right_inner_finger_joint" />
-        <group_state name="open" group="${prefix}grav_gripper">
+        <group_state name="open" group="grav_gripper">
             <joint name="${prefix}finger_width_joint" value="0.1" />
         </group_state>
-        <group_state name="closed" group="${prefix}grav_gripper">
+        <group_state name="closed" group="grav_gripper">
             <joint name="${prefix}finger_width_joint" value="0.0" />
         </group_state>
-        <end_effector name="${prefix}grav_gripper" parent_link="${prefix}flange" group="${prefix}grav_gripper" parent_group="${prefix}${name}_arm"/>
+        <end_effector name="grav_gripper" parent_link="${prefix}flange"
+            group="grav_gripper" parent_group="rizon_arm" />
         <disable_collisions link1="${prefix}grav_base_link" link2="${prefix}grav_tcp" reason="Never" />
         <disable_collisions link1="${prefix}grav_base_link" link2="${prefix}closed_fingers_tcp" reason="Never" />

File: flexiv_moveit_config/srdf/rizon_macro.srdf.xacro (robot description, xacro)
@@ -1,38 +1,41 @@
 <?xml version="1.0" encoding="UTF-8"?>
 <robot xmlns:xacro="http://www.ros.org/wiki/xacro">
-    <xacro:macro name="rizon_srdf" params="name prefix">
-        <group name="${prefix}${name}_arm">
+    <xacro:macro name="rizon_srdf" params="arm_prefix robot_sn">
+        <!-- Prefix defaults to 'arm_prefix_robot_sn' -->
+        <xacro:property name="prefix" value="${arm_prefix + robot_sn + '_'}" />
+        <group name="rizon_arm">
             <chain base_link="${prefix}base_link" tip_link="${prefix}flange" />
         </group>
-        <group_state name="${prefix}home" group="${prefix}${name}_arm">
-            <joint name="${prefix}joint1" value="0"/>
-            <joint name="${prefix}joint2" value="${-2*pi/9}"/>
-            <joint name="${prefix}joint3" value="0"/>
-            <joint name="${prefix}joint4" value="${pi/2}"/>
-            <joint name="${prefix}joint5" value="0"/>
-            <joint name="${prefix}joint6" value="${2*pi/9}"/>
-            <joint name="${prefix}joint7" value="0"/>
+        <group_state name="${prefix}home" group="rizon_arm">
+            <joint name="${prefix}joint1" value="0" />
+            <joint name="${prefix}joint2" value="${-2*pi/9}" />
+            <joint name="${prefix}joint3" value="0" />
+            <joint name="${prefix}joint4" value="${pi/2}" />
+            <joint name="${prefix}joint5" value="0" />
+            <joint name="${prefix}joint6" value="${2*pi/9}" />
+            <joint name="${prefix}joint7" value="0" />
         </group_state>
-        <virtual_joint name="virtual_joint" type="fixed" parent_frame="world" child_link="${prefix}base_link"/>
-        <disable_collisions link1="${prefix}base_link" link2="${prefix}link1" reason="Adjacent"/>
-        <disable_collisions link1="${prefix}base_link" link2="${prefix}link2" reason="Never"/>
-        <disable_collisions link1="${prefix}base_link" link2="${prefix}link3" reason="Never"/>
-        <disable_collisions link1="${prefix}base_link" link2="${prefix}link4" reason="Never"/>
-        <disable_collisions link1="${prefix}link1" link2="${prefix}link2" reason="Adjacent"/>
-        <disable_collisions link1="${prefix}link1" link2="${prefix}link3" reason="Never"/>
-        <disable_collisions link1="${prefix}link1" link2="${prefix}link4" reason="Never"/>
-        <disable_collisions link1="${prefix}link2" link2="${prefix}link3" reason="Adjacent"/>
-        <disable_collisions link1="${prefix}link2" link2="${prefix}link4" reason="Never"/>
-        <disable_collisions link1="${prefix}link2" link2="${prefix}link5" reason="Never"/>
-        <disable_collisions link1="${prefix}link3" link2="${prefix}link4" reason="Adjacent"/>
-        <disable_collisions link1="${prefix}link3" link2="${prefix}link5" reason="Never"/>
-        <disable_collisions link1="${prefix}link3" link2="${prefix}link6" reason="Never"/>
-        <disable_collisions link1="${prefix}link3" link2="${prefix}link7" reason="Never"/>
-        <disable_collisions link1="${prefix}link4" link2="${prefix}link5" reason="Adjacent"/>
-        <disable_collisions link1="${prefix}link4" link2="${prefix}link6" reason="Never"/>
-        <disable_collisions link1="${prefix}link4" link2="${prefix}link7" reason="Never"/>
-        <disable_collisions link1="${prefix}link5" link2="${prefix}link6" reason="Adjacent"/>
-        <disable_collisions link1="${prefix}link6" link2="${prefix}link7" reason="Adjacent"/>
-        <disable_collisions link1="${prefix}link7" link2="${prefix}flange" reason="Adjacent"/>
+        <virtual_joint name="virtual_joint" type="fixed" parent_frame="world"
+            child_link="${prefix}base_link" />
+        <disable_collisions link1="${prefix}base_link" link2="${prefix}link1" reason="Adjacent" />
+        <disable_collisions link1="${prefix}base_link" link2="${prefix}link2" reason="Never" />
+        <disable_collisions link1="${prefix}base_link" link2="${prefix}link3" reason="Never" />
+        <disable_collisions link1="${prefix}base_link" link2="${prefix}link4" reason="Never" />
+        <disable_collisions link1="${prefix}link1" link2="${prefix}link2" reason="Adjacent" />
+        <disable_collisions link1="${prefix}link1" link2="${prefix}link3" reason="Never" />
+        <disable_collisions link1="${prefix}link1" link2="${prefix}link4" reason="Never" />
+        <disable_collisions link1="${prefix}link2" link2="${prefix}link3" reason="Adjacent" />
+        <disable_collisions link1="${prefix}link2" link2="${prefix}link4" reason="Never" />
+        <disable_collisions link1="${prefix}link2" link2="${prefix}link5" reason="Never" />
+        <disable_collisions link1="${prefix}link3" link2="${prefix}link4" reason="Adjacent" />
+        <disable_collisions link1="${prefix}link3" link2="${prefix}link5" reason="Never" />
+        <disable_collisions link1="${prefix}link3" link2="${prefix}link6" reason="Never" />
+        <disable_collisions link1="${prefix}link3" link2="${prefix}link7" reason="Never" />
+        <disable_collisions link1="${prefix}link4" link2="${prefix}link5" reason="Adjacent" />
+        <disable_collisions link1="${prefix}link4" link2="${prefix}link6" reason="Never" />
+        <disable_collisions link1="${prefix}link4" link2="${prefix}link7" reason="Never" />
+        <disable_collisions link1="${prefix}link5" link2="${prefix}link6" reason="Adjacent" />
+        <disable_collisions link1="${prefix}link6" link2="${prefix}link7" reason="Adjacent" />
+        <disable_collisions link1="${prefix}link7" link2="${prefix}flange" reason="Adjacent" />
     </xacro:macro>
 </robot>
