Commit message: Release/Flexiv ROS 2 Jazzy v1.9 (#91)

File: flexiv_moveit_config/srdf/rizon_macro.srdf.xacro (robot description, xacro)
@@ -1,11 +1,11 @@
 <?xml version="1.0" encoding="UTF-8"?>
 <robot xmlns:xacro="http://www.ros.org/wiki/xacro">
-    <xacro:macro name="rizon_srdf" params="arm_prefix robot_sn load_mounted_ft_sensor">
+    <xacro:macro name="rizon_srdf" params="arm_prefix robot_sn load_mounted_ft_sensor use_virtual_joint:=true">
         <!-- Prefix defaults to 'arm_prefix_robot_sn' -->
         <xacro:property name="prefix" value="${arm_prefix + robot_sn + '_'}" />
-        <group name="rizon_arm">
+        <group name="${prefix}arm">
             <chain base_link="${prefix}base_link" tip_link="${prefix}flange" />
         </group>
-        <group_state name="${prefix}home" group="rizon_arm">
+        <group_state name="${prefix}home" group="${prefix}arm">
             <joint name="${prefix}joint1" value="0" />
             <joint name="${prefix}joint2" value="${-2*pi/9}" />
@@ -16,6 +16,8 @@
             <joint name="${prefix}joint7" value="0" />
         </group_state>
-        <virtual_joint name="virtual_joint" type="fixed" parent_frame="world"
-            child_link="${prefix}base_link" />
+        <xacro:if value="${use_virtual_joint}">
+            <virtual_joint name="virtual_joint" type="fixed" parent_frame="world"
+                child_link="${prefix}base_link" />
+        </xacro:if>
         <disable_collisions link1="${prefix}base_link" link2="${prefix}link1" reason="Adjacent" />
         <disable_collisions link1="${prefix}base_link" link2="${prefix}link2" reason="Never" />
